File: tinytapeout-demo.kicad_pcb (KiCad board)
At the start: 4 copper layers, 104.5 x 81 mm, 162 parts, among them J1 Conn_01x06, J10 Conn_01x02, J11 Conn_01x06, J12 613012243121, J13 613012243121, J14 613012243121, J15 USB4500-03-0-A_REVA, J16 2x20_P2.54mm_Pinheader, J17 Conn_01x03, J18 2x20_P2.54mm_Pinheader, J19 Conn_01x02, J2 Conn_01x04, J3 613012243121, J4 TT06_BREAKOUT_REVA, J5 613012243121, J6 613012243121, J7 Conn_01x02, J8 Conn_01x03, J9 Conn_01x16, Q1 DMN2005K, SW1 434121025816, SW2 434121025816, SW3 434121025816, SW4 418121270808, U1 157112V12700, U2 TLV1117LV33, U3 AP2112K-1.8, U5 W25Q32JVSS, U6 RP2040, Y1 12.0MHz

Commit message: v2.0.0 alpha, as produced for prototype run
Parts:
- removed D4: Yellow, LED_SMD:LED_0603_1608Metric
- removed J15: USB4500-03-0-A_REVA, TinyTapeout:GCT_USB4500-03-0-A_REVA
- removed R19: 510, Resistor_SMD:R_0402_1005Metric
- removed Z2ALOGO: Z2A_logo, Logos:Z2A_logo
- removed kibuzzard-63FE0D11: G***, kibuzzard-63FE0D11
- added G***: LOGO, flyingcarsfootprints:PsychoLogoSmall, B.Cu at (88.8, 77.6)
- added J20: USB_C, TinyTapeout:USB_C_Receptacle_HRO_TYPE-C-31-M-12, F.Cu at (126.5, 56.5)
- added STITCHB1: StitchingVia-0.4mmDrill, flyingcarsfootprints:StitchingVia-0.4mmDrill, F.Cu at (137.1, 67.3)
- added STITCHB1: StitchingVia-0.4mmDrill, flyingcarsfootprints:StitchingVia-0.4mmDrill, F.Cu at (154.2, 102.5)
- added STITCHB1: StitchingVia-0.4mmDrill, flyingcarsfootprints:StitchingVia-0.4mmDrill, F.Cu at (75.7, 87.8)
- added STITCHB1: StitchingVia-0.4mmDrill, flyingcarsfootprints:StitchingVia-0.4mmDrill, F.Cu at (131.1, 91.9)
- added STITCHB1: StitchingVia-0.4mmDrill, flyingcarsfootprints:StitchingVia-0.4mmDrill, F.Cu at (110.3, 130.7)
- added STITCHB1: StitchingVia-0.4mmDrill, flyingcarsfootprints:StitchingVia-0.4mmDrill, F.Cu at (86.4, 124.6)
- added STITCHB1: StitchingVia-0.4mmDrill, flyingcarsfootprints:StitchingVia-0.4mmDrill, F.Cu at (107.5, 95.3)
- added STITCHB1: StitchingVia-0.4mmDrill, flyingcarsfootprints:StitchingVia-0.4mmDrill, F.Cu at (127.1, 64.9)
- added STITCHB1: StitchingVia-0.4mmDrill, flyingcarsfootprints:StitchingVia-0.4mmDrill, F.Cu at (120.5, 130.7)
- added STITCHB1: StitchingVia-0.4mmDrill, flyingcarsfootprints:StitchingVia-0.4mmDrill, F.Cu at (88.1, 58.0)
- added STITCHB1: StitchingVia-0.4mmDrill, flyingcarsfootprints:StitchingVia-0.4mmDrill, F.Cu at (72.3, 130.7)
- added STITCHB1: StitchingVia-0.4mmDrill, flyingcarsfootprints:StitchingVia-0.4mmDrill, F.Cu at (68.2, 60.6)
- added STITCHB1: StitchingVia-0.4mmDrill, flyingcarsfootprints:StitchingVia-0.4mmDrill, F.Cu at (94.1, 124.6)
- added STITCHB1: StitchingVia-0.4mmDrill, flyingcarsfootprints:StitchingVia-0.4mmDrill, F.Cu at (147.4, 92.3)
- added STITCHB1: StitchingVia-0.4mmDrill, flyingcarsfootprints:StitchingVia-0.4mmDrill, F.Cu at (75.7, 92.7)
- added STITCHB1: StitchingVia-0.4mmDrill, flyingcarsfootprints:StitchingVia-0.4mmDrill, F.Cu at (81.9, 69.2)
- added STITCHB1: StitchingVia-0.4mmDrill, flyingcarsfootprints:StitchingVia-0.4mmDrill, F.Cu at (129.8, 85.3)
- added STITCHB1: StitchingVia-0.4mmDrill, flyingcarsfootprints:StitchingVia-0.4mmDrill, F.Cu at (123.1, 130.7)
- added STITCHB1: StitchingVia-0.4mmDrill, flyingcarsfootprints:StitchingVia-0.4mmDrill, F.Cu at (108.4, 124.2)
- added STITCHB1: StitchingVia-0.4mmDrill, flyingcarsfootprints:StitchingVia-0.4mmDrill, F.Cu at (142.9, 72.4)
- added STITCHB1: StitchingVia-0.4mmDrill, flyingcarsfootprints:StitchingVia-0.4mmDrill, F.Cu at (150.4, 66.4)
- added STITCHB1: StitchingVia-0.4mmDrill, flyingcarsfootprints:StitchingVia-0.4mmDrill, F.Cu at (154.3, 66.4)
- added STITCHB1: StitchingVia-0.4mmDrill, flyingcarsfootprints:StitchingVia-0.4mmDrill, F.Cu at (113.1, 118.8)
- added STITCHB1: StitchingVia-0.4mmDrill, flyingcarsfootprints:StitchingVia-0.4mmDrill, F.Cu at (84.7, 60.6)
- added STITCHB1: StitchingVia-0.4mmDrill, flyingcarsfootprints:StitchingVia-0.4mmDrill, F.Cu at (150.4, 119.2)
- added STITCHB1: StitchingVia-0.4mmDrill, flyingcarsfootprints:StitchingVia-0.4mmDrill, F.Cu at (108.4, 121.0)
- added STITCHB1: StitchingVia-0.4mmDrill, flyingcarsfootprints:StitchingVia-0.4mmDrill, F.Cu at (150.4, 71.4)
- added STITCHB1: StitchingVia-0.4mmDrill, flyingcarsfootprints:StitchingVia-0.4mmDrill, F.Cu at (68.6, 128.4)
- added STITCHB1: StitchingVia-0.4mmDrill, flyingcarsfootprints:StitchingVia-0.4mmDrill, F.Cu at (88.1, 63.7)
- added STITCHB1: StitchingVia-0.4mmDrill, flyingcarsfootprints:StitchingVia-0.4mmDrill, F.Cu at (92.9, 130.7)
- added STITCHB1: StitchingVia-0.4mmDrill, flyingcarsfootprints:StitchingVia-0.4mmDrill, F.Cu at (70.8, 78.5)
- added STITCHB1: StitchingVia-0.4mmDrill, flyingcarsfootprints:StitchingVia-0.4mmDrill, F.Cu at (97.7, 130.7)
- added STITCHB1: StitchingVia-0.4mmDrill, flyingcarsfootprints:StitchingVia-0.4mmDrill, F.Cu at (73.4, 60.4)
- added STITCHB1: StitchingVia-0.4mmDrill, flyingcarsfootprints:StitchingVia-0.4mmDrill, F.Cu at (131.7, 103.8)
- added STITCHB1: StitchingVia-0.4mmDrill, flyingcarsfootprints:StitchingVia-0.4mmDrill, F.Cu at (100.0, 117.2)
- added STITCHB1: StitchingVia-0.4mmDrill, flyingcarsfootprints:StitchingVia-0.4mmDrill, F.Cu at (76.4, 104.1)
- added STITCHB1: StitchingVia-0.4mmDrill, flyingcarsfootprints:StitchingVia-0.4mmDrill, F.Cu at (114.2, 96.4)
- added STITCHB1: StitchingVia-0.4mmDrill, flyingcarsfootprints:StitchingVia-0.4mmDrill, F.Cu at (77.3, 130.7)
- added STITCHB1: StitchingVia-0.4mmDrill, flyingcarsfootprints:StitchingVia-0.4mmDrill, F.Cu at (96.8, 125.0)
- added STITCHB1: StitchingVia-0.4mmDrill, flyingcarsfootprints:StitchingVia-0.4mmDrill, F.Cu at (107.5, 109.0)
- added STITCHB1: StitchingVia-0.4mmDrill, flyingcarsfootprints:StitchingVia-0.4mmDrill, F.Cu at (96.4, 58.7)
- added STITCHB1: StitchingVia-0.4mmDrill, flyingcarsfootprints:StitchingVia-0.4mmDrill, F.Cu at (127.7, 84.1)
- added STITCHB1: StitchingVia-0.4mmDrill, flyingcarsfootprints:StitchingVia-0.4mmDrill, F.Cu at (115.4, 130.7)
- added STITCHB1: StitchingVia-0.4mmDrill, flyingcarsfootprints:StitchingVia-0.4mmDrill, F.Cu at (102.7, 130.7)
- added STITCHB1: StitchingVia-0.4mmDrill, flyingcarsfootprints:StitchingVia-0.4mmDrill, F.Cu at (104.2, 119.0)
- added STITCHB1: StitchingVia-0.4mmDrill, flyingcarsfootprints:StitchingVia-0.4mmDrill, F.Cu at (73.5, 111.7)
- added STITCHB1: StitchingVia-0.4mmDrill, flyingcarsfootprints:StitchingVia-0.4mmDrill, F.Cu at (147.4, 107.2)
- added STITCHB1: StitchingVia-0.4mmDrill, flyingcarsfootprints:StitchingVia-0.4mmDrill, F.Cu at (112.9, 130.7)
- added STITCHB1: StitchingVia-0.4mmDrill, flyingcarsfootprints:StitchingVia-0.4mmDrill, F.Cu at (70.8, 86.2)
- added STITCHB1: StitchingVia-0.4mmDrill, flyingcarsfootprints:StitchingVia-0.4mmDrill, F.Cu at (75.5, 63.7)
- added STITCHB1: StitchingVia-0.4mmDrill, flyingcarsfootprints:StitchingVia-0.4mmDrill, F.Cu at (107.5, 97.6)
- added STITCHB1: StitchingVia-0.4mmDrill, flyingcarsfootprints:StitchingVia-0.4mmDrill, F.Cu at (77.0, 120.1)
- added STITCHB1: StitchingVia-0.4mmDrill, flyingcarsfootprints:StitchingVia-0.4mmDrill, F.Cu at (156.2, 110.5)
- added STITCHB1: StitchingVia-0.4mmDrill, flyingcarsfootprints:StitchingVia-0.4mmDrill, F.Cu at (122.1, 118.7)
- added STITCHB1: StitchingVia-0.4mmDrill, flyingcarsfootprints:StitchingVia-0.4mmDrill, F.Cu at (105.2, 60.4)
- added STITCHB1: StitchingVia-0.4mmDrill, flyingcarsfootprints:StitchingVia-0.4mmDrill, F.Cu at (71.6, 125.4)
- added STITCHB1: StitchingVia-0.4mmDrill, flyingcarsfootprints:StitchingVia-0.4mmDrill, F.Cu at (117.9, 130.7)
- added STITCHB1: StitchingVia-0.4mmDrill, flyingcarsfootprints:StitchingVia-0.4mmDrill, F.Cu at (111.2, 79.1)
- added STITCHB1: StitchingVia-0.4mmDrill, flyingcarsfootprints:StitchingVia-0.4mmDrill, F.Cu at (92.8, 58.1)
- added STITCHB1: StitchingVia-0.4mmDrill, flyingcarsfootprints:StitchingVia-0.4mmDrill, F.Cu at (90.3, 80.1)
- added STITCHB1: StitchingVia-0.4mmDrill, flyingcarsfootprints:StitchingVia-0.4mmDrill, F.Cu at (71.4, 90.1)
- added STITCHB1: StitchingVia-0.4mmDrill, flyingcarsfootprints:StitchingVia-0.4mmDrill, F.Cu at (87.3, 99.7)
- added STITCHB1: StitchingVia-0.4mmDrill, flyingcarsfootprints:StitchingVia-0.4mmDrill, F.Cu at (107.5, 81.0)
- added STITCHB1: StitchingVia-0.4mmDrill, flyingcarsfootprints:StitchingVia-0.4mmDrill, F.Cu at (126.3, 68.4)
- added STITCHB1: StitchingVia-0.4mmDrill, flyingcarsfootprints:StitchingVia-0.4mmDrill, F.Cu at (83.8, 101.6)
- added STITCHB1: StitchingVia-0.4mmDrill, flyingcarsfootprints:StitchingVia-0.4mmDrill, F.Cu at (154.0, 119.2)
- added STITCHB1: StitchingVia-0.4mmDrill, flyingcarsfootprints:StitchingVia-0.4mmDrill, F.Cu at (75.7, 82.6)
- added STITCHB1: StitchingVia-0.4mmDrill, flyingcarsfootprints:StitchingVia-0.4mmDrill, F.Cu at (154.3, 71.4)
- added STITCHB1: StitchingVia-0.4mmDrill, flyingcarsfootprints:StitchingVia-0.4mmDrill, F.Cu at (86.0, 97.8)
- added STITCHB1: StitchingVia-0.4mmDrill, flyingcarsfootprints:StitchingVia-0.4mmDrill, F.Cu at (68.2, 62.9)
- added STITCHB1: StitchingVia-0.4mmDrill, flyingcarsfootprints:StitchingVia-0.4mmDrill, F.Cu at (90.9, 85.4)
- added STITCHB1: StitchingVia-0.4mmDrill, flyingcarsfootprints:StitchingVia-0.4mmDrill, F.Cu at (122.1, 113.7)
- added STITCHB1: StitchingVia-0.4mmDrill, flyingcarsfootprints:StitchingVia-0.4mmDrill, F.Cu at (148.4, 130.7)
- added STITCHB1: StitchingVia-0.4mmDrill, flyingcarsfootprints:StitchingVia-0.4mmDrill, F.Cu at (147.4, 89.6)
- added STITCHB1: StitchingVia-0.4mmDrill, flyingcarsfootprints:StitchingVia-0.4mmDrill, F.Cu at (122.1, 108.9)
- added STITCHB1: StitchingVia-0.4mmDrill, flyingcarsfootprints:StitchingVia-0.4mmDrill, F.Cu at (147.4, 99.7)
- added STITCHB1: StitchingVia-0.4mmDrill, flyingcarsfootprints:StitchingVia-0.4mmDrill, F.Cu at (83.0, 89.0)
- added STITCHB1: StitchingVia-0.4mmDrill, flyingcarsfootprints:StitchingVia-0.4mmDrill, F.Cu at (107.5, 90.4)
- added STITCHB1: StitchingVia-0.4mmDrill, flyingcarsfootprints:StitchingVia-0.4mmDrill, F.Cu at (83.1, 76.7)
- added STITCHB1: StitchingVia-0.4mmDrill, flyingcarsfootprints:StitchingVia-0.4mmDrill, F.Cu at (142.4, 121.3)
- added STITCHB1: StitchingVia-0.4mmDrill, flyingcarsfootprints:StitchingVia-0.4mmDrill, F.Cu at (78.0, 60.6)
- added STITCHB1: StitchingVia-0.4mmDrill, flyingcarsfootprints:StitchingVia-0.4mmDrill, F.Cu at (66.4, 125.3)
- added STITCHB1: StitchingVia-0.4mmDrill, flyingcarsfootprints:StitchingVia-0.4mmDrill, F.Cu at (80.0, 122.5)
- added STITCHB1: StitchingVia-0.4mmDrill, flyingcarsfootprints:StitchingVia-0.4mmDrill, F.Cu at (122.5, 68.9)
- added STITCHB1: StitchingVia-0.4mmDrill, flyingcarsfootprints:StitchingVia-0.4mmDrill, F.Cu at (113.7, 76.1)
- added STITCHB1: StitchingVia-0.4mmDrill, flyingcarsfootprints:StitchingVia-0.4mmDrill, F.Cu at (146.1, 125.5)
- added STITCHB1: StitchingVia-0.4mmDrill, flyingcarsfootprints:StitchingVia-0.4mmDrill, F.Cu at (131.9, 121.3)
- added STITCHB1: StitchingVia-0.4mmDrill, flyingcarsfootprints:StitchingVia-0.4mmDrill, F.Cu at (147.4, 104.7)
- added STITCHB1: StitchingVia-0.4mmDrill, flyingcarsfootprints:StitchingVia-0.4mmDrill, F.Cu at (107.4, 100.5)
- added STITCHB1: StitchingVia-0.4mmDrill, flyingcarsfootprints:StitchingVia-0.4mmDrill, F.Cu at (71.4, 100.2)
- added STITCHB1: StitchingVia-0.4mmDrill, flyingcarsfootprints:StitchingVia-0.4mmDrill, F.Cu at (107.5, 86.7)
- added STITCHB1: StitchingVia-0.4mmDrill, flyingcarsfootprints:StitchingVia-0.4mmDrill, F.Cu at (73.4, 68.7)
- added STITCHB1: StitchingVia-0.4mmDrill, flyingcarsfootprints:StitchingVia-0.4mmDrill, F.Cu at (79.5, 71.7)
- added STITCHB1: StitchingVia-0.4mmDrill, flyingcarsfootprints:StitchingVia-0.4mmDrill, F.Cu at (136.0, 121.3)
- added STITCHB1: StitchingVia-0.4mmDrill, flyingcarsfootprints:StitchingVia-0.4mmDrill, F.Cu at (60.5, 121.5)
- added STITCHB1: StitchingVia-0.4mmDrill, flyingcarsfootprints:StitchingVia-0.4mmDrill, F.Cu at (103.8, 75.5)
- added STITCHB1: StitchingVia-0.4mmDrill, flyingcarsfootprints:StitchingVia-0.4mmDrill, F.Cu at (147.4, 94.7)
- added STITCHB1: StitchingVia-0.4mmDrill, flyingcarsfootprints:StitchingVia-0.4mmDrill, F.Cu at (87.2, 73.1)
- added STITCHB1: StitchingVia-0.4mmDrill, flyingcarsfootprints:StitchingVia-0.4mmDrill, F.Cu at (66.4, 122.5)
- added STITCHB1: StitchingVia-0.4mmDrill, flyingcarsfootprints:StitchingVia-0.4mmDrill, F.Cu at (147.4, 102.2)
- added STITCHB1: StitchingVia-0.4mmDrill, flyingcarsfootprints:StitchingVia-0.4mmDrill, F.Cu at (147.1, 120.8)
- added STITCHB1: StitchingVia-0.4mmDrill, flyingcarsfootprints:StitchingVia-0.4mmDrill, F.Cu at (147.4, 109.6)
- added STITCHB1: StitchingVia-0.4mmDrill, flyingcarsfootprints:StitchingVia-0.4mmDrill, F.Cu at (74.8, 130.7)
- added STITCHB1: StitchingVia-0.4mmDrill, flyingcarsfootprints:StitchingVia-0.4mmDrill, F.Cu at (147.4, 97.2)
- added STITCHB10: StitchingVia-0.4mmDrill, flyingcarsfootprints:StitchingVia-0.4mmDrill, F.Cu at (142.9, 80.0)
- added STITCHB11: StitchingVia-0.4mmDrill, flyingcarsfootprints:StitchingVia-0.4mmDrill, F.Cu at (142.9, 82.6)
- added STITCHB12: StitchingVia-0.4mmDrill, flyingcarsfootprints:StitchingVia-0.4mmDrill, F.Cu at (142.9, 85.1)
- added STITCHB13: StitchingVia-0.4mmDrill, flyingcarsfootprints:StitchingVia-0.4mmDrill, F.Cu at (142.9, 87.6)
- added STITCHB14: StitchingVia-0.4mmDrill, flyingcarsfootprints:StitchingVia-0.4mmDrill, F.Cu at (158.2, 61.4)
- added STITCHB15: StitchingVia-0.4mmDrill, flyingcarsfootprints:StitchingVia-0.4mmDrill, F.Cu at (158.2, 66.4)
- added STITCHB16: StitchingVia-0.4mmDrill, flyingcarsfootprints:StitchingVia-0.4mmDrill, F.Cu at (158.2, 71.4)
- added STITCHB17: StitchingVia-0.4mmDrill, flyingcarsfootprints:StitchingVia-0.4mmDrill, F.Cu at (158.2, 76.4)
- added STITCHB18: StitchingVia-0.4mmDrill, flyingcarsfootprints:StitchingVia-0.4mmDrill, F.Cu at (158.2, 81.4)
- added STITCHB19: StitchingVia-0.4mmDrill, flyingcarsfootprints:StitchingVia-0.4mmDrill, F.Cu at (158.2, 86.4)
- added STITCHB2: StitchingVia-0.4mmDrill, flyingcarsfootprints:StitchingVia-0.4mmDrill, F.Cu at (122.5, 72.9)
- added STITCHB20: StitchingVia-0.4mmDrill, flyingcarsfootprints:StitchingVia-0.4mmDrill, F.Cu at (158.2, 91.4)
- added STITCHB21: StitchingVia-0.4mmDrill, flyingcarsfootprints:StitchingVia-0.4mmDrill, F.Cu at (158.2, 96.4)
- added STITCHB22: StitchingVia-0.4mmDrill, flyingcarsfootprints:StitchingVia-0.4mmDrill, F.Cu at (158.2, 101.4)
- added STITCHB23: StitchingVia-0.4mmDrill, flyingcarsfootprints:StitchingVia-0.4mmDrill, F.Cu at (158.2, 106.4)
- added STITCHB24: StitchingVia-0.4mmDrill, flyingcarsfootprints:StitchingVia-0.4mmDrill, F.Cu at (158.2, 111.4)
- added STITCHB25: StitchingVia-0.4mmDrill, flyingcarsfootprints:StitchingVia-0.4mmDrill, F.Cu at (158.2, 116.4)
- added STITCHB26: StitchingVia-0.4mmDrill, flyingcarsfootprints:StitchingVia-0.4mmDrill, F.Cu at (158.1, 129.0)
- added STITCHB27: StitchingVia-0.4mmDrill, flyingcarsfootprints:StitchingVia-0.4mmDrill, F.Cu at (60.3, 65.4)
- added STITCHB29: StitchingVia-0.4mmDrill, flyingcarsfootprints:StitchingVia-0.4mmDrill, F.Cu at (60.3, 67.9)
- added STITCHB3: StitchingVia-0.4mmDrill, flyingcarsfootprints:StitchingVia-0.4mmDrill, F.Cu at (122.5, 76.9)
- added STITCHB30: StitchingVia-0.4mmDrill, flyingcarsfootprints:StitchingVia-0.4mmDrill, F.Cu at (60.3, 70.5)
- added STITCHB31: StitchingVia-0.4mmDrill, flyingcarsfootprints:StitchingVia-0.4mmDrill, F.Cu at (60.3, 73.0)
- added STITCHB32: StitchingVia-0.4mmDrill, flyingcarsfootprints:StitchingVia-0.4mmDrill, F.Cu at (60.3, 75.6)
- added STITCHB33: StitchingVia-0.4mmDrill, flyingcarsfootprints:StitchingVia-0.4mmDrill, F.Cu at (60.3, 78.1)
- added STITCHB34: StitchingVia-0.4mmDrill, flyingcarsfootprints:StitchingVia-0.4mmDrill, F.Cu at (60.3, 88.1)
- added STITCHB35: StitchingVia-0.4mmDrill, flyingcarsfootprints:StitchingVia-0.4mmDrill, F.Cu at (60.3, 93.6)
- added STITCHB4: StitchingVia-0.4mmDrill, flyingcarsfootprints:StitchingVia-0.4mmDrill, F.Cu at (119.9, 77.9)
- added STITCHB5: StitchingVia-0.4mmDrill, flyingcarsfootprints:StitchingVia-0.4mmDrill, F.Cu at (119.9, 74.7)
- added STITCHB6: StitchingVia-0.4mmDrill, flyingcarsfootprints:StitchingVia-0.4mmDrill, F.Cu at (119.9, 69.9)
- added STITCHB7: StitchingVia-0.4mmDrill, flyingcarsfootprints:StitchingVia-0.4mmDrill, F.Cu at (127.7, 58.1)
- added STITCHB7: StitchingVia-0.4mmDrill, flyingcarsfootprints:StitchingVia-0.4mmDrill, F.Cu at (119.9, 66.7)
- added STITCHB7: StitchingVia-0.4mmDrill, flyingcarsfootprints:StitchingVia-0.4mmDrill, F.Cu at (125.1, 55.1)
- added STITCHB7: StitchingVia-0.4mmDrill, flyingcarsfootprints:StitchingVia-0.4mmDrill, F.Cu at (125.1, 58.1)
- added STITCHB7: StitchingVia-0.4mmDrill, flyingcarsfootprints:StitchingVia-0.4mmDrill, F.Cu at (127.7, 55.1)
- added STITCHB8: StitchingVia-0.4mmDrill, flyingcarsfootprints:StitchingVia-0.4mmDrill, F.Cu at (142.9, 74.9)
- added STITCHB9: StitchingVia-0.4mmDrill, flyingcarsfootprints:StitchingVia-0.4mmDrill, F.Cu at (142.9, 77.5)
- added STITCHP3: StitchingVia-0.3mm, flyingcarsfootprints:StitchingVia-0.3mm, F.Cu at (134.6, 130.7)
- added STITCHP3: StitchingVia-0.3mm, flyingcarsfootprints:StitchingVia-0.3mm, F.Cu at (61.2, 98.5)
- added STITCHP3: StitchingVia-0.3mm, flyingcarsfootprints:StitchingVia-0.3mm, F.Cu at (76.0, 114.1)
- added STITCHP3: StitchingVia-0.3mm, flyingcarsfootprints:StitchingVia-0.3mm, F.Cu at (70.9, 119.8)
- added STITCHP3: StitchingVia-0.3mm, flyingcarsfootprints:StitchingVia-0.3mm, F.Cu at (110.1, 102.9)
- added STITCHP3: StitchingVia-0.3mm, flyingcarsfootprints:StitchingVia-0.3mm, F.Cu at (87.4, 127.7)
- added STITCHP3: StitchingVia-0.3mm, flyingcarsfootprints:StitchingVia-0.3mm, F.Cu at (61.2, 116.2)
- added STITCHP3: StitchingVia-0.3mm, flyingcarsfootprints:StitchingVia-0.3mm, F.Cu at (92.1, 118.9)
- added STITCHP3: StitchingVia-0.3mm, flyingcarsfootprints:StitchingVia-0.3mm, F.Cu at (97.3, 108.7)
- added STITCHP3: StitchingVia-0.3mm, flyingcarsfootprints:StitchingVia-0.3mm, F.Cu at (110.2, 95.6)
- added STITCHP3: StitchingVia-0.3mm, flyingcarsfootprints:StitchingVia-0.3mm, F.Cu at (61.2, 108.3)
- added STITCHP3: StitchingVia-0.3mm, flyingcarsfootprints:StitchingVia-0.3mm, F.Cu at (122.3, 79.8)
- added STITCHP3: StitchingVia-0.3mm, flyingcarsfootprints:StitchingVia-0.3mm, F.Cu at (117.2, 86.5)
- added STITCHP3: StitchingVia-0.3mm, flyingcarsfootprints:StitchingVia-0.3mm, F.Cu at (108.1, 67.4)
- added STITCHP3: StitchingVia-0.3mm, flyingcarsfootprints:StitchingVia-0.3mm, F.Cu at (110.4, 90.3)
- added STITCHP3: StitchingVia-0.3mm, flyingcarsfootprints:StitchingVia-0.3mm, F.Cu at (118.5, 87.8)
- added STITCHP3: StitchingVia-0.3mm, flyingcarsfootprints:StitchingVia-0.3mm, F.Cu at (119.8, 86.5)
- added STITCHP3: StitchingVia-0.3mm, flyingcarsfootprints:StitchingVia-0.3mm, F.Cu at (71.3, 114.1)
- added STITCHP3: StitchingVia-0.3mm, flyingcarsfootprints:StitchingVia-0.3mm, F.Cu at (118.5, 85.2)
- SW4: value 418121270808 -> 193-8MSR; footprint TinyTapeout:418121270808 -> TinyTapeout:GENERIC_PIANO_8DIP
- moved FID1 99.8 mm to (157.5, 118.5)
- moved C25 63.0 mm to (88.5, 68.5), turned to -90 degrees
- moved C16 62.6 mm to (146.0, 66.4), turned to -90 degrees
- moved REF** 62.5 mm to (87.5, 68.5)
- moved C21 61.4 mm to (90.0, 68.5), turned to -90 degrees
- moved C17 59.0 mm to (146.0, 71.0)
- moved R42 57.6 mm to (104.0, 103.0)
- moved REF** 52.7 mm to (81.4, 118.5)
- moved R43 52.4 mm to (104.0, 100.5), turned to 0 degrees
- moved R51 52.1 mm to (130.1, 81.7), turned to 180 degrees
- moved R44 51.8 mm to (104.0, 98.0), turned to 0 degrees
- moved R40 51.4 mm to (108.0, 71.0), turned to -90 degrees
- moved U5 50.9 mm to (113.5, 71.8)
- moved J11 50.9 mm to (112.1, 72.7)
- moved R35 50.6 mm to (108.0, 73.5), turned to 90 degrees
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Connections:
- J16 pad 1: unconnected-(J16-Pad1) -> GND
- J18 pad 1: unconnected-(J18-Pad1) -> out6
- J9 pad 10: ctrl_sel_inc -> res1
- J9 pad 11: GND -> res2
- J9 pad 12: res1 -> res3
- J9 pad 13: res2 -> GND
- J9 pad 14: res3 -> RPIO29
- J9 pad 16: RPIO29 -> +5V
- J9 pad 2: +5V -> +3V3
- J9 pad 4: +3V3 -> +1V8
- J9 pad 6: +1V8 -> ctrl_ena
- J9 pad 7: GND -> ~{ctrl_sel_rst}
- J9 pad 8: ctrl_ena -> ctrl_sel_inc
- J9 pad 9: ~{ctrl_sel_rst} -> GND
- U6 pad 4: ctrl_sel_inc -> ~{ctrl_sel_rst}
- U6 pad 5: ctrl_ena -> ctrl_sel_inc
- U6 pad 6: ~{ctrl_sel_rst} -> ctrl_ena
Routing:
- net +3V3: track 0.00 -> 656.1 mm, vias 0 -> 62
- net out1: track 0.00 -> 190.7 mm, vias 0 -> 8
- net uio3: track 0.00 -> 182.1 mm, vias 0 -> 7
- net uio5: track 0.00 -> 178.0 mm, vias 0 -> 6
- net in2: track 0.00 -> 175.4 mm, vias 0 -> 9
- net GND: track 0.00 -> 171.2 mm, vias 0 -> 89
- net out7: track 0.00 -> 168.6 mm, vias 0 -> 8
- net uio6: track 0.00 -> 168.1 mm, vias 0 -> 6
- net uio4: track 0.00 -> 167.1 mm, vias 0 -> 6
- net out4: track 0.00 -> 166.4 mm, vias 0 -> 9
- net in5: track 0.00 -> 162.5 mm, vias 0 -> 8
- net out3: track 0.00 -> 162.0 mm, vias 0 -> 4
- net +5V: track 0.00 -> 158.9 mm, vias 0 -> 9
- net in7: track 0.00 -> 158.5 mm, vias 0 -> 7
- net in1: track 0.00 -> 153.0 mm, vias 0 -> 6
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Other:
- board size 104.5 x 81 mm -> 99.5 x 78 mm
- board text added: "Design by Pat Deegan"
- board text added: "Designed by"
- board text added: "Open Source Hardware"
- board text added: "R29"
- board text added: "RS1"
- board text added: "RS2"
- board text added: "RS3"
- board text added: "TinyTapeout 06+ Demo Board"
- board text added: "TinyTapeout 06+ Demoboard"
- board text added: "psychogenic.com"
- board text added: "v2.0"
- board text added: "v2.0.0"
- board text removed: "3v3 GND 3v3 GND bi6 bi7 bi4 bi5 bi2 bi3 bi1 GND GND 1v8 3v3 1v8 3v3 GND GND GND ot7 bi0 ot5 GND GND ot6 ot3 ot4 ot1 ot2 GND ot0 1v8 GND 1v8 GND 3v3 GND 3v3 GND"
- board text removed: "CSB"
- board text removed: "Designed by Pat Deegan https://psychogenic.com"
- board text removed: "HK SPI"
- board text removed: "IN PWR"
- board text removed: "Input"
- board text removed: "OFF"
- board text removed: "ON"
- board text removed: "P29"
- board text removed: "Power and RP2040 data"
- board text removed: "RP2040 FLASH"
- board text removed: "SDI"
- board text removed: "SDO"
- board text removed: "TT04+ Carrier"
- board text removed: "TinyTapeout 4+ Demo Board"
- board text removed: "TinyTapeout 4+ Demoboard"
- board text removed: "UCK"
- board text removed: "cEN GND c++ m33 m37 m35 1v8 cRS GND GND xCK xRS cCK cCS GND cD0 cD1 GPIO 3v3 GND hSO m00 hCS hSI GND hCK uCK pCK GND GND pRS in0 in1 in2 in3 in4 in5 in6 in7 GND"
- board text removed: "m00"
- board text removed: "m33"
- board text removed: "m35"
- board text removed: "m37"
- board text removed: "v1.2"
- board text removed: "v1.2.4"

Commit message: minor fab cleanups
Parts:
- renumbered REF** to OSHWBADGE1, REF** to OSHWLOGO2, G*** to PSYLOGO1, PSYLOGO to PSYLOGO2, TTLOGO to TTLOGO1, REF** to Z2ALOGO2

Commit message: renamed JLC field to LCSC, minor tweaks to BOM
Parts:
- renumbered REF** to TTLOGO2
Connections:
- J16 pad 1: GND -> unconnected-(J16-Pad1)
- J18 pad 1: out6 -> unconnected-(J18-Pad1)
