File: tinytapeout-demo.kicad_pcb (KiCad board)
At the start: 4 copper layers, 99.5 x 78 mm, 319 parts, among them J1 Conn_01x06, J10 Conn_01x02, J11 Conn_01x06, J12 613012243121, J13 613012243121, J14 613012243121, J16 2x20_P2.54mm_Pinheader, J17 Conn_01x03, J18 2x20_P2.54mm_Pinheader, J19 Conn_01x02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

Commit message: v2.1.0, TT07
Other:
- board text added: "v2.1"
- board text removed: "v2.0"
Changed lines of the file:
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@@
 		)
 	)
-	(gr_text "v2.0"
+	(gr_text "v2.1"
 		(at 122.5392 67.3 90)
 		(layer "B.SilkS")

Commit message: efabless logo
Parts:
- added REF**: Logo, Logos:ef_logo_graphical, F.Cu at (153.4, 66.0)
- added REF**: Logo, Logos:ef_logo, F.Cu at (153.4, 70.4)
- moved TTLOGO1 1.07 mm to (150.1, 82.4)
Other:
- board text added: "(C) 2025 TinyTapeout"
- board text added: "v2.1.1"
- board text removed: "(C) 2024 TinyTapeout"
- board text removed: "v2.1.0"
