File: tinytapeout-demo.kicad_sch (KiCad schematic)
At the start: 129 parts, among them J1 Conn_01x06, J12 613012243121, J13 613012243121, J14 613012243121, J15 USB4500-03-0-A_REVA, J16 2x20_P2.54mm_Pinheader, J17 Conn_01x03, J18 2x20_P2.54mm_Pinheader, J19 Conn_01x02, J2 Conn_01x04, J3 613012243121, J4 TT06_BREAKOUT_REVA, J5 613012243121, J6 613012243121, J7 Conn_01x02, J8 Conn_01x03, J9 Conn_01x16, Q1 DMN2005K, SW1 434121025816, SW2 434121025816, SW3 434121025816, SW4 418121270808, U1 157112V12700, U2 TLV1117LV33, U3 AP2112K-1.8

Commit message: first remap of pcb and global delete of all routing
Other:
- note added: "USER-FACING CHANGES from TT04 * top header (J9) shorter, pin changes * no demoboard MUX in the way of low out nibble * more comfortable input DIP (rocker or piano, TBD) All RP2040 pin mappings for I/O are the same. All PMOD connectors are the same. Project reset and ASIC MUX pins have moved, but will be transparent for SDK users. MAJOR Changes from TT04 * carrier board new size and pinout * analo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"
- title: Tiny Tapeout 4/5 Demo Board -> Tiny Tapeout 06+ Demo Board
Changed lines of the file:
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@@
 	(paper "A3")
 	(title_block
-		(title "Tiny Tapeout 4/5 Demo Board")
-		(date "2024-04-12")
-		(rev "1.2.2")
+		(title "Tiny Tapeout 06+ Demo Board")
+		(date "2024-08-10")
+		(rev "2.0.0")
 		(company "Psychogenic Technologies")
-		(comment 1 "(C) 2023, 2024 Pat Deegan")
+		(comment 1 "(C) 2024 Pat Deegan")
 	)
 	(junction
@@
 		)
 	)
+	(text "USER-FACING CHANGES from TT04\n * top header (J9) shorter, pin changes\n * no demoboard MUX in the way of low out nibble\n * more comfortable input DIP (rocker or \n   piano, TBD)\n\nAll RP2040 pin mappings for I/O are the same.  \nAll PMOD connectors are the same.\nProject reset and ASIC MUX pins have moved, \nbut will be transparent for SDK users.\n\nMAJOR Changes from TT04\n * carrier board new size and pinout\n * analog terminations on DB, but interfacing\n   happens on carrier (though a jumper from\n   u.fl to ADC on RPIO29 pin top header)\n * no demoboard MUXing of RP2040 I/O\n * nothing caravel related (osc, flash, etc)\n"
+		(exclude_from_sim no)
+		(at 339.344 42.926 0)
+		(effects
+			(font
+				(size 1.75 1.75)
+			)
+			(justify left)
+		)
+	)

Commit message: v2.0.0 alpha, as produced for prototype run
Parts:
- removed D4: Yellow, LED_SMD:LED_0603_1608Metric, symbol Device:LED_Small
- removed J15: USB4500-03-0-A_REVA, TinyTapeout:GCT_USB4500-03-0-A_REVA, symbol TinyTapeout:USB4500-03-0-A_REVA
- removed R19: 510, Resistor_SMD:R_0402_1005Metric, symbol Device:R_Small
- added J20: USB_C, TinyTapeout:USB_C_Receptacle_HRO_TYPE-C-31-M-12, symbol TinyTapeout:USB_C_Receptacle_USB2.0
- SW4: value 418121270808 -> 193-8MSR; footprint TinyTapeout:418121270808 -> TinyTapeout:GENERIC_PIANO_8DIP; Characteristics 8 POS SPST DIP -> 8 POS SPST DIP PIANO; DigikeyPN (none) -> CT3100CT-ND; JLC C2842673 -> C3293170; MPN 418121270808 -> DSPV08LSGET; MPN_ALT 219-8MST -> 2.54-8P TPCB
Connections:
- net +1V8: now also J9.4 (Pin_4); no longer J9.6 (Pin_6)
- net +3V3: now also J9.2 (Pin_2); no longer J9.4 (Pin_4)
- net +5V: now also J9.16 (Pin_16); no longer J9.2 (Pin_2)
- net CC1: now also J20.A5 (CC1)
- net CC2: now also J20.B5 (CC2)
- net GND: now also J9.13 (Pin_13), J9.9 (Pin_9), J20.A1 (GND), J20.A12 (GND), J20.B1 (GND), J20.B12 (GND); no longer J9.11 (Pin_11), J9.7 (Pin_7)
- net RPIO29: now also J9.14 (Pin_14); no longer J9.16 (Pin_16)
- net VBUS: now also J20.A4 (VBUS), J20.A9 (VBUS), J20.B4 (VBUS), J20.B9 (VBUS)
- net ctrl_ena: now also J9.6 (Pin_6); no longer J9.8 (Pin_8)
- net ctrl_sel_inc: now also J9.8 (Pin_8); no longer J9.10 (Pin_10)
- net res1: now also J9.10 (Pin_10); no longer J9.12 (Pin_12)
- net res2: now also J9.11 (Pin_11); no longer J9.13 (Pin_13)
- net res3: now also J9.12 (Pin_12); no longer J9.14 (Pin_14)
- net usb_d+: now also J20.A6 (D+), J20.B6 (D+)
- net usb_d-: now also J20.A7 (D-), J20.B7 (D-)
- net ~{ctrl_sel_rst}: now also J9.7 (Pin_7); no longer J9.9 (Pin_9)
- net at C3.1, R16.1: now also J20.S1 (SHIELD)
Other:
- note added: "TT06+ Demoboard: complete re-organization, support for TT06+ new carrier pinout. For users, main difference is the new piano DIP input and the fact no MUX is in the way on demoboards."
- note added: "Tiny Tapeout 06+ Demo Board"
- note added: "i2c eeprom on carrier 2: SDA1 3: SCL1"
- note removed: "Tiny Tapeout 06+ Demo Board: PRELIMINARY"
- moved on the sheet: C3, J9, R16

Commit message: minor fab cleanups
Parts:
- C44, C45, C46, C47: Characteristics (none) -> 33pF 0402
- FB1: Characteristics (none) -> FERRITE BEAD 120R 0603
- J12, J13, J14, J3, J5, J6: Characteristics (none) -> 2x6 female pin header 100mil
- R16: Characteristics (none) -> 1M 0603
Changed lines of the file:
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@@
 			)
 		)
-		(property "Characteristics" ""
+		(property "Characteristics" "2x6 female pin header 100mil"
 			(at 132.08 251.46 0)
 			(effects
@@
 			)
 		)
-		(property "Characteristics" ""
+		(property "Characteristics" "2x6 female pin header 100mil"
 			(at 276.86 251.46 0)
 			(effects
@@
 			)
 		)
-		(property "Characteristics" ""
+		(property "Characteristics" "2x6 female pin header 100mil"
 			(at 185.42 251.46 0)
 			(effects
@@
 			)
 		)
-		(property "Characteristics" ""
+		(property "Characteristics" "33pF 0402"
 			(at 147.32 78.74 0)
 			(effects
@@
 			)
 		)
-		(property "Characteristics" ""
+		(property "Characteristics" "2x6 female pin header 100mil"
 			(at 40.64 251.46 0)
 			(effects
@@
 			)
 		)
-		(property "Characteristics" ""
+		(property "Characteristics" "2x6 female pin header 100mil"
 			(at 86.36 251.46 0)
 			(effects
@@
 			)
 		)
-		(property "Characteristics" ""
+		(property "Characteristics" "33pF 0402"
 			(at 146.05 49.53 0)
 			(effects
@@
 			)
 		)
-		(property "Characteristics" ""
+		(property "Characteristics" "33pF 0402"
 			(at 157.48 78.74 0)
 			(effects
@@
 			)
 		)
-		(property "Characteristics" ""
+		(property "Characteristics" "2x6 female pin header 100mil"
 			(at 228.6 251.46 0)
 			(effects
@@
 			)
 		)
-		(property "Characteristics" ""
+		(property "Characteristics" "FERRITE BEAD 120R 0603 "
 			(at 161.29 31.75 0)
 			(effects
@@
 			)
 		)
-		(property "Characteristics" ""
+		(property "Characteristics" "33pF 0402"
 			(at 156.21 46.99 0)
 			(effects
@@
 			(at 100.33 81.28 0)
 			(effects
+				(font
+					(size 1.27 1.27)
+				)
+				(hide yes)
+			)
+		)
+		(property "Characteristics" "1M 0603"
+			(at 100.33 81.28 0)
+			(effects

Commit message: renamed JLC field to LCSC, minor tweaks to BOM
Parts:
- C1, C11, C15, C17, C25, C48, C49, C5, C57, C59, C61, C9: JLC C5673 -> (none); LCSC (none) -> C5673
- C10: JLC C86816 -> (none); LCSC (none) -> C86816
- C12, C13, C14, C2, C23, C24, C26, C4, C56, C58, C60, C8: JLC C100072 -> (none); LCSC (none) -> C100072
- C16, C21: JLC C962136 -> (none); LCSC (none) -> C962136; MPN_ALT GRT188R61C106KE13J -> GRT188R61C106KE13J
- C44, C45, C46, C47: JLC C107005 -> (none); LCSC (none) -> C107005
- C6, C7: JLC C237493 -> (none); LCSC (none) -> C237493
- D1, D2, D3: JLC C72038 -> (none); LCSC (none) -> C72038
- D5, D6: JLC C6961594 -> (none); LCSC (none) -> C6961594
- F1: JLC C1884490 -> (none); LCSC (none) -> C1884490
- FB1: Characteristics FERRITE BEAD 120R 0603 -> FERRITE BEAD 120R 0603; JLC C2649119 -> (none); LCSC (none) -> C2649119
- J12, J13, J14, J3, J5, J6: JLC C6147817 -> (none); LCSC (none) -> C6147817
- J16, J18: JLC C3294478 -> (none); LCSC (none) -> C3294478
- Q1: JLC C2891732 -> (none); LCSC (none) -> C2891732
- R1, R10, R11, R13, R14, R2, R3, R4, R5, R6: JLC C202394 -> (none); LCSC (none) -> C202394
- R12, R30, R31, R32, R42, R43, R44, R45, R46, R47, R48, R51, R52, R53, R54, R55, R8, R9: JLC C471764 -> (none); LCSC (none) -> C471764
- R15: JLC C138040 -> (none); LCSC (none) -> C138040
- R16: JLC C858907 -> (none); LCSC (none) -> C858907
- R17, R18, R22, R23, R24, R25, R26, R27, R28, R29: JLC C276273 -> (none); LCSC (none) -> C276273
- R20, R21: JLC C138073 -> (none); LCSC (none) -> C138073
- R41, R50: JLC C4271317 -> (none); LCSC (none) -> C4271317
- R49: JLC C95177 -> (none); LCSC (none) -> C95177
- R7: JLC C327139 -> (none); LCSC (none) -> C327139
- SW1, SW2, SW3: JLC C5525525 -> (none); LCSC (none) -> C329185
- SW4: JLC C3293170 -> (none); LCSC (none) -> C3293170
- U1: Characteristics 7 SEGMENT COMMON CATHODE -> 7 SEGMENT COMMON CATHODE; JLC C6976938 -> (none); LCSC (none) -> C6976938
- U2: JLC C15578 -> (none); LCSC (none) -> C15578
- U3: JLC C176944 -> (none); LCSC (none) -> C176944
