File: rp2040.kicad_sch (KiCad schematic)
At the start: 25 parts, among them J10 Conn_01x02, J11 Conn_01x06, U5 W25Q32JVSS, U6 RP2040, Y1 12.0MHz

Commit message: v3p5 pcba BOM tweaks
Parts:
- U5: Characteristics (none) -> RP2040 FLASH
Changed lines of the file:
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@@
 			)
 		)
-		(property "Characteristics" ""
+		(property "Characteristics" "RP2040 FLASH"
 			(at 50.8 180.34 0)
 			(effects
+				(font
+					(size 1.27 1.27)
+				)
+				(hide yes)
+			)
+		)
+		(property "Variant" ""
+			(at 50.8 180.34 0)
+			(effects
+				(font
+					(size 1.27 1.27)
+				)
+				(hide yes)
+			)
+		)
+		(property "MPN_ALT" ""
+			(at 50.8 180.34 0)
+			(effects

Commit message: JLC MPNs
Parts:
- C29, C30: JLC (none) -> C541341
- C31, C33, C34, C35, C36, C38, C39, C40, C41: JLC (none) -> C100072
- C32, C37: JLC (none) -> C5673
- R34, R35, R36, R38, R39, R40: JLC (none) -> C471764
- R37: JLC (none) -> C202394
- U5: JLC (none) -> C82344
- U6: JLC (none) -> C3227924
- Y1: JLC (none) -> C6098259; MPN_ALT (none) -> ABM8W-12.0000MHZ-8-D1X-T3
Changed lines of the file:
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@@
 			)
 		)
+		(property "JLC" "C541341"
+			(at 55.88 109.22 0)
+			(effects
+				(font
+					(size 1.27 1.27)
+				)
+				(hide yes)
+			)
+		)
 		(pin "1"
 		)
@@
 			)
 		)
-		(property "JLC" ""
+		(property "JLC" "C471764"
 			(at 80.01 167.64 0)
 			(effects
@@
 			)
 		)
+		(property "JLC" "C100072"
+			(at 119.38 177.8 0)
+			(effects
+				(font
+					(size 1.27 1.27)
+				)
+				(hide yes)
+			)
+		)
 		(pin "1"
 		)
@@
 			)
 		)
+		(property "JLC" "C3227924"
+			(at 109.22 91.44 0)
+			(effects
+				(font
+					(size 1.27 1.27)
+				)
+				(hide yes)
+			)
+		)
 		(pin "1"
 		)
@@
 			)
 		)
+		(property "JLC" "C100072"
+			(at 119.38 167.64 0)
+			(effects
+				(font
+					(size 1.27 1.27)
+				)
+				(hide yes)
+			)
+		)
 		(pin "1"
 		)
@@
 			)
 		)
+		(property "JLC" "C100072"
+			(at 129.54 177.8 0)
+			(effects
+				(font
+					(size 1.27 1.27)
+				)
+				(hide yes)
+			)
+		)
 		(pin "1"
 		)
@@
 			)
 		)
+		(property "JLC" "C100072"
+			(at 157.48 175.26 0)
+			(effects
+				(font
+					(size 1.27 1.27)
+				)
+				(hide yes)
+			)
+		)
 		(pin "1"
 		)
@@
 			)
 		)
+		(property "JLC" "C202394"
+			(at 73.66 109.22 0)
+			(effects
+				(font
+					(size 1.27 1.27)
+				)
+				(hide yes)
+			)
+		)
 		(pin "1"
 		)
@@
 			)
 		)
-		(property "JLC" ""
+		(property "JLC" "C471764"
 			(at 25.4 170.18 0)
 			(effects
@@
 			)
 		)
+		(property "JLC" "C471764"
+			(at 73.66 48.26 0)
+			(effects
+				(font
+					(size 1.27 1.27)
+				)
+				(hide yes)
+			)
+		)
 		(pin "1"
 		)
@@
 			)
 		)
+		(property "JLC" "C100072"
+			(at 129.54 167.64 0)
+			(effects
+				(font
+					(size 1.27 1.27)
+				)
+				(hide yes)
+			)
+		)
 		(pin "1"
 		)
@@
 			)
 		)
+		(property "JLC" "C100072"
+			(at 109.22 167.64 0)
+			(effects
+				(font
+					(size 1.27 1.27)
+				)
+				(hide yes)
+			)
+		)
 		(pin "1"
 		)
@@
 			)
 		)
+		(property "JLC" "C6098259"
+			(at 60.96 104.14 0)
+			(effects
+				(font
+					(size 1.27 1.27)
+				)
+				(hide yes)
+			)
+		)
+		(property "MPN_ALT" "ABM8W-12.0000MHZ-8-D1X-T3"
+			(at 60.96 104.14 0)
+			(effects
+				(font
+					(size 1.27 1.27)
+				)
+				(hide yes)
+			)
+		)
 		(pin "1"
 		)
@@
 			)
 		)
+		(property "JLC" "C5673"
+			(at 96.52 43.18 0)
+			(effects
+				(font
+					(size 1.27 1.27)
+				)
+				(hide yes)
+			)
+		)
 		(pin "1"
 		)
@@
 			)
 		)
+		(property "JLC" "C541341"
+			(at 55.88 99.06 0)
+			(effects
+				(font
+					(size 1.27 1.27)
+				)
+				(hide yes)
+			)
+		)
 		(pin "1"
 		)
@@
 			)
 		)
+		(property "JLC" "C82344"
+			(at 50.8 180.34 0)
+			(effects
+				(font
+					(size 1.27 1.27)
+				)
+				(hide yes)
+			)
+		)
 		(pin "1"
 		)
@@
 			)
 		)
+		(property "JLC" "C5673"
+			(at 124.46 43.18 0)
+			(effects
+				(font
+					(size 1.27 1.27)
+				)
+				(hide yes)
+			)
+		)
 		(pin "1"
 		)
@@
 			)
 		)
-		(property "JLC" ""
+		(property "JLC" "C471764"
 			(at 73.66 167.64 0)
 			(effects
@@
 			)
 		)
+		(property "JLC" "C100072"
+			(at 109.22 177.8 0)
+			(effects
+				(font
+					(size 1.27 1.27)
+				)
+				(hide yes)
+			)
+		)
 		(pin "1"
 		)
@@
 			)
 		)
-		(property "JLC" ""
+		(property "JLC" "C471764"
 			(at 86.36 167.64 0)
 			(effects
@@
 			)
 		)
-		(property "JLC" ""
+		(property "JLC" "C100072"
 			(at 57.15 167.64 0)
 			(effects
@@
 			)
 		)
-		(property "JLC" ""
+		(property "JLC" "C471764"
 			(at 67.31 167.64 0)
 			(effects
@@
 			(at 149.86 175.26 0)
 			(effects
+				(font
+					(size 1.27 1.27)
+				)
+				(hide yes)
+			)
+		)
+		(property "JLC" "C100072"
+			(at 149.86 175.26 0)
+			(effects

Commit message: PMOD header DNP swap/fix
Parts:
- C30: MPN_ALT (none) -> 0402N6R0D500CT
Changed lines of the file:
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@@
+			)
+		)
+		(property "MPN_ALT" "0402N6R0D500CT"
+			(at 55.88 109.22 0)
+			(effects
+				(font
+					(size 1.27 1.27)
+				)
+				(hide yes)
 			)
 		)

Commit message: v1.2.3, TT05 run plus mod to brighten 1v8 LED (pwr via 3v3, gate fet using 1v8)
Other:
- note removed: "in2 GPIO11, 1RTS out0 GPIO 5, 1RX in7 GPIO20, 1TX out1 GPIO6, 1CTS"
- title: RP2040 Basic Support -> Tiny Tapeout 4/5 Demo Board
Changed lines of the file:
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@@
 	(paper "A4")
 	(title_block
-		(title "RP2040 Basic Support")
-		(date "2023-11-22")
-		(rev "1.0.3")
+		(title "Tiny Tapeout 4/5 Demo Board")
+		(date "2024-04-12")
+		(rev "1.2.2")
 		(company "Psychogenic Technologies")
-		(comment 1 "(C) 2023 Pat Deegan")
+		(comment 1 "(C) 2023, 2024 Pat Deegan")
 	)
 	(junction
@@
 		(effects
 			(font
-				(size 1.27 1.27)
-			)
-			(justify left bottom)
-		)
-	)
-	(text " in2 GPIO11, 1RTS\nout0 GPIO 5, 1RX \nin7 GPIO20, 1TX\nout1 GPIO6, 1CTS"
-		(exclude_from_sim no)
-		(at 162.56 78.74 0)
-		(effects
-			(font

Commit message: renamed JLC field to LCSC, minor tweaks to BOM
Parts:
- C29, C30: JLC C541341 -> (none); LCSC (none) -> C541341
- C31, C33, C34, C35, C36, C38, C39, C40, C41: JLC C100072 -> (none); LCSC (none) -> C100072
- C32, C37: JLC C5673 -> (none); LCSC (none) -> C5673
- R34, R35, R36, R38, R39, R40: JLC C471764 -> (none); LCSC (none) -> C471764
- R37: JLC C202394 -> (none); LCSC (none) -> C202394
- U5: JLC C82344 -> (none); LCSC (none) -> C82344
- U6: JLC C3227924 -> (none); LCSC (none) -> C2040
- Y1: JLC C6098259 -> (none); LCSC (none) -> C5288803
