File: rp2350.kicad_sch (KiCad schematic)
At the start: 32 parts, among them J15 Conn_01x03, U3 RP2350-QFN80, U4 W25Q32JVSS, Y1 12.0MHz

Commit message: re-annotated entire schem
Parts:
- renumbered C26 to C30, C27 to C31, C28 to C32, C29 to C33, C30 to C34, C31 to C35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
